File: BusLink.kicad_pcb (KiCad board)
At the start: 4 copper layers, 0 parts

Commit message: setting up heirarchy
Parts:
- added J1: DE9_Pins, Connector_Dsub:DSUB-9_Pins_Horizontal_P2.77x2.84mm_EdgePinOffset9.90mm_Housed_MountingHolesOffset11.32mm, F.Cu at (93.4, 98.5)
- added J2: USB_C_Receptacle_USB2.0_14P, Connector_USB:USB_C_Receptacle_GCT_USB4110, F.Cu at (126.4, 106.0)
- added U1: STM32H723VETx, Package_QFP:LQFP-100_14x14mm_P0.5mm, F.Cu at (108.0, 110.0)
- added U2: USB3300-EZK, Package_DFN_QFN:QFN-32-1EP_5x5mm_P0.5mm_EP3.45x3.45mm, F.Cu at (122.8, 114.3)
