File: can.kicad_sch (KiCad schematic)
At the start: 0 parts

Commit message: working on power supplies and CAN
Parts:
- added C1, C3: 1u, Capacitor_SMD:C_0603_1608Metric, symbol Device:C
- added C2, C4: 100n, Capacitor_SMD:C_0603_1608Metric, symbol Device:C
- added U3, U4: SN65HVD230, Package_SO:SOIC-8_3.9x4.9mm_P1.27mm, symbol Interface_CAN_LIN:SN65HVD230
Connections:
- net CAN0_HI: now also U3.7 (CANH)
- net CAN0_LO: now also U3.6 (CANL)
- net CAN1_HI: now also U4.7 (CANH)
- net CAN1_LO: now also U4.6 (CANL)
- net GND: now also C1.2, C2.2, C3.2, C4.2, U3.2 (GND), U3.8 (Rs), U4.2 (GND), U4.8 (Rs)
- new net +3V3: C1.1, C2.1, C3.1, C4.1, U3.3 (VCC), U4.3 (VCC)
- new net CAN0_RX: U3.4 (R)
- new net CAN0_TX: U3.1 (D)
- new net CAN1_RX: U4.4 (R)
- new net CAN1_TX: U4.1 (D)
- no-connect marks 0 -> 2
