File: pwr.kicad_sch (KiCad schematic)
At the start: 10 parts, among them U5 XL1509-3.3, U7 AP2112K-1.8

Commit message: added inductor selection
Parts:
- L1: footprint (none) -> Inductor_SMD:L_Sunlord_SWPA4030S
Changed lines of the file:
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@@
 			)
 		)
-		(property "Footprint" ""
+		(property "Footprint" "Inductor_SMD:L_Sunlord_SWPA4030S"
 			(at 139.7 78.74 0)
 			(effects
